File: USB_soundcard_board/USB_soundcard_board.kicad_pcb (KiCad board)
At the start: 2 copper layers, 85.6 x 55.9 mm, 104 parts, among them IC1 USBLC6-2SC6, IC2 CP2112-F03-GMR, IC3 CP2615-A02-GMR, IC4 USBLC6-2SC6, IC5 AP2112K-1.8, J1 TT04_BREAKOUT_REVB, U1 Raspberry Pi Pico

Commit message: Post-prototype tweaks in USB board schematic
Parts:
- C27, C34: value 3p -> 2p7
- C29, C30, L3: value DNP -> 0R
- L1: value 663n -> 650n
- L2: value 191n -> 200n
- moved C10 212.7 mm to (180.6, 79.2)
- moved C12 212.7 mm to (187.7, 88.0)
- moved C15 212.7 mm to (146.6, 81.8)
- moved C20 212.7 mm to (157.9, 118.5)
- moved C25 212.7 mm to (148.1, 97.5)
- moved C35 212.7 mm to (157.9, 72.7)
- moved C36 212.7 mm to (157.9, 113.4)
- moved C6 212.7 mm to (170.0, 79.2)
- moved F1 212.7 mm to (143.2, 87.7)
- moved FB1 212.7 mm to (172.6, 80.0)
- moved IC1 212.7 mm to (170.0, 79.2)
- moved IC2 212.7 mm to (187.0, 81.1)
- moved IC4 212.7 mm to (180.6, 79.2)
- moved IC5 212.7 mm to (146.6, 84.8)
- moved JP3 212.7 mm to (176.4, 80.0)
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